File: trunk/pcb/zif_socket.sch (KiCad schematic (older format))
At the start: 5 parts, among them P1 CONN_5, U1 PIC18F4550, U2 PIC12F675, U3 PIC16F628A, U4 PIC18F2550

Commit message: created zif-socket pcb
git-svn-id: https://usbpicprog.svn.sourceforge.net/svnroot/usbpicprog@367 29735491-9d32-0410-b17f-ed4c7e910dea
Parts:
- removed U1: PIC18F4550, symbol PIC18F4550
- removed U2: PIC12F675, symbol PIC12F675
- removed U3: PIC16F628A, symbol PIC16F628A
- removed U4: PIC18F2550, symbol PIC18F2550
- added P1: DIL40, symbol DIL40
- added P2: dsPIC40P, symbol CONN_5
- added P3: dsPIC28P, symbol CONN_5
- added P4: dsPIC18P, symbol CONN_5
- added P5: PIC28-40P, symbol CONN_5
- added P7: PIC12F_8-14P, symbol CONN_5
- added P8: PIC10F_8P, symbol CONN_5
- P6: renamed from P1; value CONN_5 -> PIC18P
Connections:
- net labels added: GND10F, GND18, GND40, MCLR12F, MCLR40, PGC12F, PGC18, PGCdsPIC28, PGCdsPIC40, PGD10F, PGD12F, PGD18, PGD40, PGDdsPIC18, PGDdsPIC28, PGDdsPIC40, VDD18, VDD40
- net labels removed: MCLR, PGC, PGD, VDD, VSS
- wire segments 38 -> 53
Other:
- moved on the sheet: P6
