File: trunk/pcb/usbpicprog.sch (KiCad schematic (older format))
At the start: 36 parts, among them J1 USB_CONN, P1 CONN_5, P2 CONN_5, Q1 BS170, Q2 BS170, Q3 TSM2301CX, U1 PIC18F2550, X1 8MHz

Commit message: modified schematic for PIC24 and dsPIC33 devices, PCB not yet finished, will be released as v0.3
git-svn-id: https://usbpicprog.svn.sourceforge.net/svnroot/usbpicprog@377 29735491-9d32-0410-b17f-ed4c7e910dea
Parts:
- added R10, R11: 470, symbol R
- added R9: 1k, symbol R
- R4, R5: value 100 -> 470
Connections:
- wire segments 108 -> 119
Other:
- moved on the sheet: R4, R5
Changed lines of the file:
@@
-EESchema Schematic File Version 1
-LIBS:power,usb-b,device,conn,linear,regul,74xx,cmos4000,adc-dac,memory,xilinx,special,microcontrollers,dsp,microchip,analog_switches,motorola,texas,intel,audio,interface,digital-audio,philips,display,cypress,siliconi,contrib,valves,.\usbpicprog.cache
+EESchema Schematic File Version 2
+LIBS:power,device,conn,linear,regul,74xx,cmos4000,adc-dac,memory,xilinx,special,microcontrollers,dsp,microchip,analog_switches,motorola,texas,intel,audio,interface,digital-audio,philips,display,cypress,siliconi,contrib,valves,.\usbpicprog.cache
 EELAYER 23  0
 EELAYER END
@@
 Title "Usbpicprog"
 Date "23 oct 2007"
-Rev "0.2"
+Rev "0.3"
 Comp "Usb Slim and Basic Pic In Circuit PROGrammer"
 Comment1 "http://usbpicprog.sourceforge.net"
@@
 Comment4 ""
 $EndDescr
+Connection ~ 8600 3200
+Wire Wire Line
+	8600 3700 8600 3200
+Connection ~ 8400 3100
+Wire Wire Line
+	8200 3100 8750 3100
+Wire Wire Line
+	8750 3100 8750 2150
+Wire Wire Line
+	8750 2150 10150 2150
+Wire Wire Line
+	8600 4200 8600 4400
 Wire Wire Line
 	8000 2050 7950 2050
@@
 	3750 4800 3750 4850
 Wire Wire Line
-	9500 2350 8900 2350
+	7700 3300 7100 3300
 Wire Wire Line
 	10150 1950 8900 1950
 Wire Wire Line
-	10000 2350 10050 2350
-Wire Wire Line
-	10050 2350 10050 2250
-Wire Wire Line
-	10050 2250 10150 2250
+	8200 3300 8250 3300
+Wire Wire Line
+	8250 3300 8250 3200
 Wire Wire Line
 	9600 3350 10150 3350
@@
 	9600 3250 10150 3250
 Wire Wire Line
-	10000 2150 10150 2150
-Wire Wire Line
-	9500 2150 8900 2150
+	7700 3100 7100 3100
 Wire Wire Line
 	5450 1400 4850 1400
@@
 Wire Wire Line
 	8400 2050 10150 2050
+Wire Wire Line
+	7250 2600 7250 2650
+Wire Wire Line
+	8400 4200 8400 4300
+Wire Wire Line
+	8400 4300 7150 4300
+Wire Wire Line
+	8400 3100 8400 3700
+Wire Wire Line
+	8250 3200 8850 3200
+Wire Wire Line
+	8850 3200 8850 2250
+Wire Wire Line
+	8850 2250 10150 2250
+Wire Wire Line
+	8600 4400 7150 4400
+$Comp
+L R R11
+U 1 1 49096B01
+P 8600 3950
+F 0 "R11" V 8680 3950 50  0000 C C
+F 1 "470" V 8600 3950 50  0000 C C
+	1    8600 3950
+	-1   0    0    1
+$EndComp
+$Comp
+L R R10
+U 1 1 49096ACD
+P 8400 3950
+F 0 "R10" V 8480 3950 50  0000 C C
+F 1 "470" V 8400 3950 50  0000 C C
+	1    8400 3950
+	-1   0    0    1
+$EndComp
+$Comp
+L R R9
+U 1 1 49096A85
+P 7250 2350
+F 0 "R9" V 7330 2350 50  0000 C C
+F 1 "1k" V 7250 2350 50  0000 C C
+	1    7250 2350
+	-1   0    0    1
+$EndComp
 $Comp
 L DIODE D9
@@
 Text Label 7500 5800 0    60   ~
 VDD_CTL
-Text Label 7250 2100 0    60   ~
+Text Label 7250 2650 0    60   ~
 VDD_CTL
 $Comp
@@
 	1    0    0    -1
 $EndComp
-Text Label 8900 2350 0    60   ~
+Text Label 7100 3300 0    60   ~
 PGC
-Text Label 8900 2150 0    60   ~
+Text Label 7100 3100 0    60   ~
 PGD
 Text Label 8900 1950 0    60   ~
@@
 L R R5
 U 1 1 466D175B
-P 9750 2350
-F 0 "R5" V 9830 2350 50  0000 C C
-F 1 "100" V 9750 2350 50  0000 C C
-	1    9750 2350
+P 7950 3300
+F 0 "R5" V 8030 3300 50  0000 C C
+F 1 "470" V 7950 3300 50  0000 C C
+	1    7950 3300
 	0    1    1    0
 $EndComp
@@
 L R R4
 U 1 1 466D175A
-P 9750 2150
-F 0 "R4" V 9830 2150 50  0000 C C
-F 1 "100" V 9750 2150 50  0000 C C
-	1    9750 2150
+P 7950 3100
+F 0 "R4" V 8030 3100 50  0000 C C
+F 1 "470" V 7950 3100 50  0000 C C
+	1    7950 3100
 	0    1    1    0
 $EndComp

Commit message: added extra functionality to the pcb; 5V on VPP and voltage dividers on PGD and PGC
git-svn-id: https://usbpicprog.svn.sourceforge.net/svnroot/usbpicprog@621 29735491-9d32-0410-b17f-ed4c7e910dea
Parts:
- added Q4: BS170, symbol FET_N
- added Q5: TSM2301CX, symbol FET_P
- added R12, R13: 100k, symbol R
- added R14: 1k, symbol R
Connections:
- wire segments 119 -> 131
Other:
- moved on the sheet: R2, R3

Commit message: some last value changes in the pcb (0.3) almost ready to release!
git-svn-id: https://usbpicprog.svn.sourceforge.net/svnroot/usbpicprog@663 29735491-9d32-0410-b17f-ed4c7e910dea
Parts:
- C2, C3: value 15p -> 22p
- D5: value LED -> RED
- D6: value LED -> YELLOW
- D7: value LED -> GREEN
- R10, R11: value 470 -> 1k
- R6, R7, R8: value 150 -> 470
Changed lines of the file:
@@
-EESchema Schematic File Version 1
-LIBS:power,device,conn,linear,regul,74xx,cmos4000,adc-dac,memory,xilinx,special,microcontrollers,dsp,microchip,analog_switches,motorola,texas,intel,audio,interface,digital-audio,philips,display,cypress,siliconi,contrib,valves,./usbpicprog.cache
+EESchema Schematic File Version 2
+LIBS:power,device,conn,linear,regul,74xx,cmos4000,adc-dac,memory,xilinx,special,microcontrollers,dsp,microchip,analog_switches,motorola,texas,intel,audio,interface,digital-audio,philips,display,cypress,siliconi,contrib,valves,.\usbpicprog.cache
 EELAYER 23  0
 EELAYER END
@@
 P 8600 3950
 F 0 "R11" V 8680 3950 50  0000 C C
-F 1 "470" V 8600 3950 50  0000 C C
+F 1 "1k" V 8600 3950 50  0000 C C
 	1    8600 3950
 	-1   0    0    1
@@
 P 8400 3950
 F 0 "R10" V 8480 3950 50  0000 C C
-F 1 "470" V 8400 3950 50  0000 C C
+F 1 "1k" V 8400 3950 50  0000 C C
 	1    8400 3950
 	-1   0    0    1
@@
 P 1850 3700
 F 0 "R8" V 1930 3700 50  0000 C C
-F 1 "150" V 1850 3700 50  0000 C C
+F 1 "470" V 1850 3700 50  0000 C C
 	1    1850 3700
 	-1   0    0    1
@@
 P 1550 3700
 F 0 "R7" V 1630 3700 50  0000 C C
-F 1 "150" V 1550 3700 50  0000 C C
+F 1 "470" V 1550 3700 50  0000 C C
 	1    1550 3700
 	-1   0    0    1
@@
 P 1250 3700
 F 0 "R6" V 1330 3700 50  0000 C C
-F 1 "150" V 1250 3700 50  0000 C C
+F 1 "470" V 1250 3700 50  0000 C C
 	1    1250 3700
 	1    0    0    -1
@@
 P 1850 4250
 F 0 "D7" H 1850 4350 50  0000 C C
-F 1 "LED" H 1850 4150 50  0000 C C
+F 1 "GREEN" H 1850 4150 50  0000 C C
 	1    1850 4250
 	0    1    1    0
@@
 P 1550 4250
 F 0 "D6" H 1550 4350 50  0000 C C
-F 1 "LED" H 1550 4150 50  0000 C C
+F 1 "YELLOW" H 1550 4150 50  0000 C C
 	1    1550 4250
 	0    1    1    0
@@
 P 1250 4250
 F 0 "D5" H 1250 4350 50  0000 C C
-F 1 "LED" H 1250 4150 50  0000 C C
+F 1 "RED" H 1250 4150 50  0000 C C
 	1    1250 4250
 	0    1    1    0
@@
 P 4350 6600
 F 0 "C3" H 4400 6700 50  0000 L C
-F 1 "15p" H 4400 6500 50  0000 L C
+F 1 "22p" H 4400 6500 50  0000 L C
 	1    4350 6600
 	1    0    0    -1
@@
 P 3400 6600
 F 0 "C2" H 3450 6700 50  0000 L C
-F 1 "15p" H 3450 6500 50  0000 L C
+F 1 "22p" H 3450 6500 50  0000 L C
 	1    3400 6600
 	1    0    0    -1

Commit message: added voltage check on VPP
git-svn-id: https://usbpicprog.svn.sourceforge.net/svnroot/usbpicprog@664 29735491-9d32-0410-b17f-ed4c7e910dea
Parts:
- added R15: 100k, symbol R
- added R16: 47k, symbol R
- D5: value RED -> WR
- D6: value YELLOW -> RD
- D7: value GREEN -> ON
Connections:
- wire segments 131 -> 137
Changed lines of the file:
@@
 EESchema Schematic File Version 2
-LIBS:power,device,conn,linear,regul,74xx,cmos4000,adc-dac,memory,xilinx,special,microcontrollers,dsp,microchip,analog_switches,motorola,texas,intel,audio,interface,digital-audio,philips,display,cypress,siliconi,contrib,valves,.\usbpicprog.cache
+LIBS:power,device,conn,linear,regul,74xx,cmos4000,adc-dac,memory,xilinx,special,microcontrollers,dsp,microchip,analog_switches,motorola,texas,intel,audio,interface,digital-audio,philips,display,cypress,siliconi,contrib,valves,./usbpicprog.cache
 EELAYER 23  0
 EELAYER END
@@
 Sheet 1 1
 Title "Usbpicprog"
-Date "17 apr 2009"
+Date "23 may 2009"
 Rev "0.3"
 Comp "Usb Slim and Basic Pic In Circuit PROGrammer"
@@
 Comment4 ""
 $EndDescr
+Text Label 9000 5150 0    60   ~
+VPP
+Wire Wire Line
+	7150 4100 8050 4100
+Wire Wire Line
+	8050 4100 8050 5850
+Connection ~ 9000 5850
+Wire Wire Line
+	8050 5850 9000 5850
+Wire Wire Line
+	9000 5800 9000 5900
 Wire Wire Line
 	7150 4200 8150 4200
@@
 Wire Wire Line
 	9550 4900 9600 4900
+Wire Wire Line
+	9000 5300 9000 5150
+Wire Wire Line
+	9000 6400 9000 6500
+$Comp
+L VSS #PWR01
+U 1 1 4A17C526
+P 9000 6500
+F 0 "#PWR01" H 9000 6500 30  0001 C C
+F 1 "VSS" H 9000 6430 30  0000 C C
+	1    9000 6500
+	1    0    0    -1
+$EndComp
+$Comp
+L R R16
+U 1 1 4A17C51E
+P 9000 6150
+F 0 "R16" V 9080 6150 50  0000 C C
+F 1 "47k" V 9000 6150 50  0000 C C
+	1    9000 6150
+	-1   0    0    1
+$EndComp
+$Comp
+L R R15
+U 1 1 4A17C513
+P 9000 5550
+F 0 "R15" V 9080 5550 50  0000 C C
+F 1 "100k" V 9000 5550 50  0000 C C
+	1    9000 5550
+	-1   0    0    1
+$EndComp
 Text Label 10100 5450 0    60   ~
 VPP
@@
 $EndComp
 $Comp
-L VDD #PWR01
+L VDD #PWR02
 U 1 1 49E8D2D9
 P 10050 4450
-F 0 "#PWR01" H 10050 4550 30  0001 C C
+F 0 "#PWR02" H 10050 4550 30  0001 C C
 F 1 "VDD" H 10050 4560 30  0000 C C
 	1    10050 4450
@@
 $EndComp
 $Comp
-L VSS #PWR02
+L VSS #PWR03
 U 1 1 466D3886
 P 8450 2550
-F 0 "#PWR02" H 8450 2550 30  0001 C C
+F 0 "#PWR03" H 8450 2550 30  0001 C C
 F 1 "VSS" H 8450 2480 30  0000 C C
 	1    8450 2550
@@
 $EndComp
 $Comp
-L VDD #PWR03
+L VDD #PWR04
 U 1 1 466D3882
 P 9150 3100
-F 0 "#PWR03" H 9150 3200 30  0001 C C
+F 0 "#PWR04" H 9150 3200 30  0001 C C
 F 1 "VDD" H 9150 3210 30  0000 C C
 	1    9150 3100
@@
 $EndComp
 $Comp
-L VSS #PWR04
+L VSS #PWR05
 U 1 1 466D3881
 P 9150 3600
-F 0 "#PWR04" H 9150 3600 30  0001 C C
+F 0 "#PWR05" H 9150 3600 30  0001 C C
 F 1 "VSS" H 9150 3530 30  0000 C C
 	1    9150 3600
@@
 $EndComp
 $Comp
-L VDD #PWR05
+L VDD #PWR06
 U 1 1 466D387C
 P 3350 4800
-F 0 "#PWR05" H 3350 4900 30  0001 C C
+F 0 "#PWR06" H 3350 4900 30  0001 C C
 F 1 "VDD" H 3350 4910 30  0000 C C
 	1    3350 4800
@@
 $EndComp
 $Comp
-L VSS #PWR06
+L VSS #PWR07
 U 1 1 466D387B
 P 3350 5300
-F 0 "#PWR06" H 3350 5300 30  0001 C C
+F 0 "#PWR07" H 3350 5300 30  0001 C C
 F 1 "VSS" H 3350 5230 30  0000 C C
 	1    3350 5300
@@
 $EndComp
 $Comp
-L VDD #PWR07
+L VDD #PWR08
 U 1 1 466D3879
 P 3750 4800
-F 0 "#PWR07" H 3750 4900 30  0001 C C
+F 0 "#PWR08" H 3750 4900 30  0001 C C
 F 1 "VDD" H 3750 4910 30  0000 C C
 	1    3750 4800
@@
 $EndComp
 $Comp
-L VSS #PWR08
+L VSS #PWR09
 U 1 1 466D3878
 P 3750 5300
-F 0 "#PWR08" H 3750 5300 30  0001 C C
+F 0 "#PWR09" H 3750 5300 30  0001 C C
 F 1 "VSS" H 3750 5230 30  0000 C C
 	1    3750 5300
@@
 VPP
 $Comp
-L VDD #PWR09
+L VDD #PWR010
 U 1 1 466D37B0
 P 7950 1050
-F 0 "#PWR09" H 7950 1150 30  0001 C C
+F 0 "#PWR010" H 7950 1150 30  0001 C C
 F 1 "VDD" H 7950 1160 30  0000 C C
 	1    7950 1050
@@
 VPP_SELF
 $Comp
-L VDD #PWR010
+L VDD #PWR011
 U 1 1 466D3740
 P 9850 3150
-F 0 "#PWR010" H 9850 3250 30  0001 C C
+F 0 "#PWR011" H 9850 3250 30  0001 C C
 F 1 "VDD" H 9850 3260 30  0000 C C
 	1    9850 3150
@@
 $EndComp
 $Comp
-L VSS #PWR011
+L VSS #PWR012
 U 1 1 466D36FC
 P 10100 3600
-F 0 "#PWR011" H 10100 3600 30  0001 C C
+F 0 "#PWR012" H 10100 3600 30  0001 C C
 F 1 "VSS" H 10100 3530 30  0000 C C
 	1    10100 3600
@@
 LED1
 $Comp
-L VDD #PWR012
+L VDD #PWR013
 U 1 1 466D3690
 P 1550 3350
-F 0 "#PWR012" H 1550 3450 30  0001 C C
+F 0 "#PWR013" H 1550 3450 30  0001 C C
 F 1 "VDD" H 1550 3460 30  0000 C C
 	1    1550 3350
@@
 P 1850 4250
 F 0 "D7" H 1850 4350 50  0000 C C
-F 1 "GREEN" H 1850 4150 50  0000 C C
+F 1 "ON" H 1850 4150 50  0000 C C
 	1    1850 4250
 	0    1    1    0
@@
 P 1550 4250
 F 0 "D6" H 1550 4350 50  0000 C C
-F 1 "YELLOW" H 1550 4150 50  0000 C C
+F 1 "RD" H 1550 4150 50  0000 C C
 	1    1550 4250
 	0    1    1    0
@@
 P 1250 4250
 F 0 "D5" H 1250 4350 50  0000 C C
-F 1 "RED" H 1250 4150 50  0000 C C
+F 1 "WR" H 1250 4150 50  0000 C C
 	1    1250 4250
 	0    1    1    0
@@
 Pump1
 $Comp
-L VSS #PWR013
+L VSS #PWR014
 U 1 1 466D3412
 P 4350 6900
-F 0 "#PWR013" H 4350 6900 30  0001 C C
+F 0 "#PWR014" H 4350 6900 30  0001 C C
 F 1 "VSS" H 4350 6830 30  0000 C C
 	1    4350 6900
@@
 $EndComp
 $Comp
-L VSS #PWR014
+L VSS #PWR015
 U 1 1 466D340F
 P 3400 6900
-F 0 "#PWR014" H 3400 6900 30  0001 C C
+F 0 "#PWR015" H 3400 6900 30  0001 C C
 F 1 "VSS" H 3400 6830 30  0000 C C
 	1    3400 6900
@@
 VPP
 $Comp
-L VDD #PWR015
+L VDD #PWR016
 U 1 1 466D33A4
 P 4350 4750
-F 0 "#PWR015" H 4350 4850 30  0001 C C
+F 0 "#PWR016" H 4350 4850 30  0001 C C
 F 1 "VDD" H 4350 4860 30  0000 C C
 	1    4350 4750
@@
 $EndComp
 $Comp
-L VSS #PWR016
+L VSS #PWR017
 U 1 1 466D338E
 P 4350 5400
-F 0 "#PWR016" H 4350 5400 30  0001 C C
+F 0 "#PWR017" H 4350 5400 30  0001 C C
 F 1 "VSS" H 4350 5330 30  0000 C C
 	1    4350 5400
@@
 $EndComp
 $Comp
-L VSS #PWR017
+L VSS #PWR018
 U 1 1 466D337E
 P 4350 5650
-F 0 "#PWR017" H 4350 5650 30  0001 C C
+F 0 "#PWR018" H 4350 5650 30  0001 C C
 F 1 "VSS" H 4350 5580 30  0000 C C
 	1    4350 5650
@@
 D+
 $Comp
-L VDD #PWR018
+L VDD #PWR019
 U 1 1 466D3343
 P 1350 1500
-F 0 "#PWR018" H 1350 1600 30  0001 C C
+F 0 "#PWR019" H 1350 1600 30  0001 C C
 F 1 "VDD" H 1350 1610 30  0000 C C
 	1    1350 1500
@@
 $EndComp
 $Comp
-L VDD #PWR019
+L VDD #PWR020
 U 1 1 466D3340
 P 950 1250
-F 0 "#PWR019" H 950 1350 30  0001 C C
+F 0 "#PWR020" H 950 1350 30  0001 C C
 F 1 "VDD" H 950 1360 30  0000 C C
 	1    950  1250
@@
 $EndComp
 $Comp
-L VSS #PWR020
+L VSS #PWR021
 U 1 1 466D3322
 P 2250 1900
-F 0 "#PWR020" H 2250 1900 30  0001 C C
+F 0 "#PWR021" H 2250 1900 30  0001 C C
 F 1 "VSS" H 2250 1830 30  0000 C C
 	1    2250 1900
@@
 $EndComp
 $Comp
-L VSS #PWR021
+L VSS #PWR022
 U 1 1 466D331E
 P 1350 1800
-F 0 "#PWR021" H 1350 1800 30  0001 C C
+F 0 "#PWR022" H 1350 1800 30  0001 C C
 F 1 "VSS" H 1350 1730 30  0000 C C
 	1    1350 1800
@@
 $EndComp
 $Comp
-L VSS #PWR022
+L VSS #PWR023
 U 1 1 466D3319
 P 1350 1900
-F 0 "#PWR022" H 1350 1900 30  0001 C C
+F 0 "#PWR023" H 1350 1900 30  0001 C C
 F 1 "VSS" H 1350 1830 30  0000 C C
 	1    1350 1900
@@
 $EndComp
 $Comp
-L VSS #PWR023
+L VSS #PWR024
 U 1 1 466D330A
 P 950 1750
-F 0 "#PWR023" H 950 1750 30  0001 C C
+F 0 "#PWR024" H 950 1750 30  0001 C C
 F 1 "VSS" H 950 1680 30  0000 C C
 	1    950  1750
@@
 $EndComp
 $Comp
-L VSS #PWR024
+L VSS #PWR025
 U 1 1 466D196D
 P 6850 2150
-F 0 "#PWR024" H 6850 2150 30  0001 C C
+F 0 "#PWR025" H 6850 2150 30  0001 C C
 F 1 "VSS" H 6850 2080 30  0000 C C
 	1    6850 2150
@@
 $EndComp
 $Comp
-L VSS #PWR025
+L VSS #PWR026
 U 1 1 466D196B
 P 6500 2250
-F 0 "#PWR025" H 6500 2250 30  0001 C C
+F 0 "#PWR026" H 6500 2250 30  0001 C C
 F 1 "VSS" H 6500 2180 30  0000 C C
 	1    6500 2250
@@
 $EndComp
 $Comp
-L VSS #PWR026
+L VSS #PWR027
 U 1 1 466D1967
 P 5300 2850
-F 0 "#PWR026" H 5300 2850 30  0001 C C
+F 0 "#PWR027" H 5300 2850 30  0001 C C
 F 1 "VSS" H 5300 2780 30  0000 C C
 	1    5300 2850
@@
 VPP_CTL
 $Comp
-L VDD #PWR027
+L VDD #PWR028
 U 1 1 466D18DB
 P 2650 1300
-F 0 "#PWR027" H 2650 1400 30  0001 C C
+F 0 "#PWR028" H 2650 1400 30  0001 C C
 F 1 "VDD" H 2650 1410 30  0000 C C
 	1    2650 1300
@@
 $EndComp
 $Comp
-L VSS #PWR028
+L VSS #PWR029
 U 1 1 466D18CA
 P 4250 2200
-F 0 "#PWR028" H 4250 2200 30  0001 C C
+F 0 "#PWR029" H 4250 2200 30  0001 C C
 F 1 "VSS" H 4250 2130 30  0000 C C
 	1    4250 2200
@@
 $EndComp
 $Comp
-L VSS #PWR029
+L VSS #PWR030
 U 1 1 466D1791
 P 10100 2500
-F 0 "#PWR029" H 10100 2500 30  0001 C C
+F 0 "#PWR030" H 10100 2500 30  0001 C C
 F 1 "VSS" H 10100 2430 30  0000 C C
 	1    10100 2500

Commit message: fixed BIG error in PCB v0.3 / implemented initialization of newly used pins in firmware
git-svn-id: https://usbpicprog.svn.sourceforge.net/svnroot/usbpicprog@701 29735491-9d32-0410-b17f-ed4c7e910dea
Parts:
- added D10: 1n4148, symbol DIODE
Connections:
- wire segments 137 -> 138

Commit message: I screwed up.... :( fixed diode !
git-svn-id: https://usbpicprog.svn.sourceforge.net/svnroot/usbpicprog@702 29735491-9d32-0410-b17f-ed4c7e910dea
Parts:
- removed Q5: TSM2301CX, symbol FET_P
Connections:
- wire segments 138 -> 135
Changed lines of the file:
@@
 $EndDescr
 Wire Wire Line
-	10500 5450 10650 5450
+	10050 4900 10200 4900
 Wire Wire Line
 	9000 6400 9000 6500
@@
 	9000 5300 9000 5150
 Wire Wire Line
-	9550 4900 9600 4900
+	9550 4900 9650 4900
 Connection ~ 6650 1400
 Wire Wire Line
@@
 	7250 1500 7500 1500
 Wire Wire Line
-	10100 5450 10050 5450
-Wire Wire Line
-	10050 4450 10050 4550
-Wire Wire Line
-	10050 5450 10050 5250
-Wire Wire Line
 	9050 4900 8150 4900
 Wire Wire Line
@@
 L DIODE D10
 U 1 1 4A447726
-P 10300 5450
-F 0 "D10" H 10300 5550 40  0000 C C
-F 1 "1n4148" H 10300 5350 40  0000 C C
-	1    10300 5450
+P 9850 4900
+F 0 "D10" H 9850 5000 40  0000 C C
+F 1 "1n4148" H 9850 4800 40  0000 C C
+	1    9850 4900
 	1    0    0    -1
 $EndComp
@@
 	-1   0    0    1
 $EndComp
-Text Label 10650 5450 0    60   ~
+Text Label 10200 4900 0    60   ~
 VPP
 $Comp
@@
 	0    -1   -1   0
 $EndComp
-$Comp
-L FET_P Q5
-U 1 1 49E8D2DA
-P 9900 4900
-F 0 "Q5" H 9803 5150 70  0000 C C
-F 1 "TSM2301CX" H 9753 4653 60  0000 C C
-	1    9900 4900
-	1    0    0    1
-$EndComp
-$Comp
-L VDD #PWR02
-U 1 1 49E8D2D9
-P 10050 4450
-F 0 "#PWR02" H 10050 4550 30  0001 C C
-F 1 "VDD" H 10050 4560 30  0000 C C
-	1    10050 4450
-	1    0    0    -1
-$EndComp
 Text Label 7250 2650 0    60   ~
 VDD_CTL
@@
 $EndComp
 $Comp
-L VSS #PWR03
+L VSS #PWR02
 U 1 1 466D3886
 P 8450 2550
-F 0 "#PWR03" H 8450 2550 30  0001 C C
+F 0 "#PWR02" H 8450 2550 30  0001 C C
 F 1 "VSS" H 8450 2480 30  0000 C C
 	1    8450 2550
@@
 $EndComp
 $Comp
-L VDD #PWR04
+L VDD #PWR03
 U 1 1 466D3882
 P 9150 3100
-F 0 "#PWR04" H 9150 3200 30  0001 C C
+F 0 "#PWR03" H 9150 3200 30  0001 C C
 F 1 "VDD" H 9150 3210 30  0000 C C
 	1    9150 3100
@@
 $EndComp
 $Comp
-L VSS #PWR05
+L VSS #PWR04
 U 1 1 466D3881
 P 9150 3600
-F 0 "#PWR05" H 9150 3600 30  0001 C C
+F 0 "#PWR04" H 9150 3600 30  0001 C C
 F 1 "VSS" H 9150 3530 30  0000 C C
 	1    9150 3600
@@
 $EndComp
 $Comp
-L VDD #PWR06
+L VDD #PWR05
 U 1 1 466D387C
 P 3350 4800
-F 0 "#PWR06" H 3350 4900 30  0001 C C
+F 0 "#PWR05" H 3350 4900 30  0001 C C
 F 1 "VDD" H 3350 4910 30  0000 C C
 	1    3350 4800
@@
 $EndComp
 $Comp
-L VSS #PWR07
+L VSS #PWR06
 U 1 1 466D387B
 P 3350 5300
-F 0 "#PWR07" H 3350 5300 30  0001 C C
+F 0 "#PWR06" H 3350 5300 30  0001 C C
 F 1 "VSS" H 3350 5230 30  0000 C C
 	1    3350 5300
@@
 $EndComp
 $Comp
-L VDD #PWR08
+L VDD #PWR07
 U 1 1 466D3879
 P 3750 4800
-F 0 "#PWR08" H 3750 4900 30  0001 C C
+F 0 "#PWR07" H 3750 4900 30  0001 C C
 F 1 "VDD" H 3750 4910 30  0000 C C
 	1    3750 4800
@@
 $EndComp
 $Comp
-L VSS #PWR09
+L VSS #PWR08
 U 1 1 466D3878
 P 3750 5300
-F 0 "#PWR09" H 3750 5300 30  0001 C C
+F 0 "#PWR08" H 3750 5300 30  0001 C C
 F 1 "VSS" H 3750 5230 30  0000 C C
 	1    3750 5300
@@
 VPP
 $Comp
-L VDD #PWR010
+L VDD #PWR09
 U 1 1 466D37B0
 P 7950 1050
-F 0 "#PWR010" H 7950 1150 30  0001 C C
+F 0 "#PWR09" H 7950 1150 30  0001 C C
 F 1 "VDD" H 7950 1160 30  0000 C C
 	1    7950 1050
@@
 VPP_SELF
 $Comp
-L VDD #PWR011
+L VDD #PWR010
 U 1 1 466D3740
 P 9850 3150
-F 0 "#PWR011" H 9850 3250 30  0001 C C
+F 0 "#PWR010" H 9850 3250 30  0001 C C
 F 1 "VDD" H 9850 3260 30  0000 C C
 	1    9850 3150
@@
 $EndComp
 $Comp
-L VSS #PWR012
+L VSS #PWR011
 U 1 1 466D36FC
 P 10100 3600
-F 0 "#PWR012" H 10100 3600 30  0001 C C
+F 0 "#PWR011" H 10100 3600 30  0001 C C
 F 1 "VSS" H 10100 3530 30  0000 C C
 	1    10100 3600
@@
 LED1
 $Comp
-L VDD #PWR013
+L VDD #PWR012
 U 1 1 466D3690
 P 1550 3350
-F 0 "#PWR013" H 1550 3450 30  0001 C C
+F 0 "#PWR012" H 1550 3450 30  0001 C C
 F 1 "VDD" H 1550 3460 30  0000 C C
 	1    1550 3350
@@
 Pump1
 $Comp
-L VSS #PWR014
+L VSS #PWR013
 U 1 1 466D3412
 P 4350 6900
-F 0 "#PWR014" H 4350 6900 30  0001 C C
+F 0 "#PWR013" H 4350 6900 30  0001 C C
 F 1 "VSS" H 4350 6830 30  0000 C C
 	1    4350 6900
@@
 $EndComp
 $Comp
-L VSS #PWR015
+L VSS #PWR014
 U 1 1 466D340F
 P 3400 6900
-F 0 "#PWR015" H 3400 6900 30  0001 C C
+F 0 "#PWR014" H 3400 6900 30  0001 C C
 F 1 "VSS" H 3400 6830 30  0000 C C
 	1    3400 6900
@@
 VPP
 $Comp
-L VDD #PWR016
+L VDD #PWR015
 U 1 1 466D33A4
 P 4350 4750
-F 0 "#PWR016" H 4350 4850 30  0001 C C
+F 0 "#PWR015" H 4350 4850 30  0001 C C
 F 1 "VDD" H 4350 4860 30  0000 C C
 	1    4350 4750
@@
 $EndComp
 $Comp
-L VSS #PWR017
+L VSS #PWR016
 U 1 1 466D338E
 P 4350 5400
-F 0 "#PWR017" H 4350 5400 30  0001 C C
+F 0 "#PWR016" H 4350 5400 30  0001 C C
 F 1 "VSS" H 4350 5330 30  0000 C C
 	1    4350 5400
@@
 $EndComp
 $Comp
-L VSS #PWR018
+L VSS #PWR017
 U 1 1 466D337E
 P 4350 5650
-F 0 "#PWR018" H 4350 5650 30  0001 C C
+F 0 "#PWR017" H 4350 5650 30  0001 C C
 F 1 "VSS" H 4350 5580 30  0000 C C
 	1    4350 5650
@@
 D+
 $Comp
-L VDD #PWR019
+L VDD #PWR018
 U 1 1 466D3343
 P 1350 1500
-F 0 "#PWR019" H 1350 1600 30  0001 C C
+F 0 "#PWR018" H 1350 1600 30  0001 C C
 F 1 "VDD" H 1350 1610 30  0000 C C
 	1    1350 1500
@@
 $EndComp
 $Comp
-L VDD #PWR020
+L VDD #PWR019
 U 1 1 466D3340
 P 950 1250
-F 0 "#PWR020" H 950 1350 30  0001 C C
+F 0 "#PWR019" H 950 1350 30  0001 C C
 F 1 "VDD" H 950 1360 30  0000 C C
 	1    950  1250
@@
 $EndComp
 $Comp
-L VSS #PWR021
+L VSS #PWR020
 U 1 1 466D3322
 P 2250 1900
-F 0 "#PWR021" H 2250 1900 30  0001 C C
+F 0 "#PWR020" H 2250 1900 30  0001 C C
 F 1 "VSS" H 2250 1830 30  0000 C C
 	1    2250 1900
@@
 $EndComp
 $Comp
-L VSS #PWR022
+L VSS #PWR021
 U 1 1 466D331E
 P 1350 1800
-F 0 "#PWR022" H 1350 1800 30  0001 C C
+F 0 "#PWR021" H 1350 1800 30  0001 C C
 F 1 "VSS" H 1350 1730 30  0000 C C
 	1    1350 1800
@@
 $EndComp
 $Comp
-L VSS #PWR023
+L VSS #PWR022
 U 1 1 466D3319
 P 1350 1900
-F 0 "#PWR023" H 1350 1900 30  0001 C C
+F 0 "#PWR022" H 1350 1900 30  0001 C C
 F 1 "VSS" H 1350 1830 30  0000 C C
 	1    1350 1900
@@
 $EndComp
 $Comp
-L VSS #PWR024
+L VSS #PWR023
 U 1 1 466D330A
 P 950 1750
-F 0 "#PWR024" H 950 1750 30  0001 C C
+F 0 "#PWR023" H 950 1750 30  0001 C C
 F 1 "VSS" H 950 1680 30  0000 C C
 	1    950  1750
@@
 $EndComp
 $Comp
-L VSS #PWR025
+L VSS #PWR024
 U 1 1 466D196D
 P 6850 2150
-F 0 "#PWR025" H 6850 2150 30  0001 C C
+F 0 "#PWR024" H 6850 2150 30  0001 C C
 F 1 "VSS" H 6850 2080 30  0000 C C
 	1    6850 2150
@@
 $EndComp
 $Comp
-L VSS #PWR026
+L VSS #PWR025
 U 1 1 466D196B
 P 6500 2250
-F 0 "#PWR026" H 6500 2250 30  0001 C C
+F 0 "#PWR025" H 6500 2250 30  0001 C C
 F 1 "VSS" H 6500 2180 30  0000 C C
 	1    6500 2250
@@
 $EndComp
 $Comp
-L VSS #PWR027
+L VSS #PWR026
 U 1 1 466D1967
 P 5300 2850
-F 0 "#PWR027" H 5300 2850 30  0001 C C
+F 0 "#PWR026" H 5300 2850 30  0001 C C
 F 1 "VSS" H 5300 2780 30  0000 C C
 	1    5300 2850
@@
 VPP_CTL
 $Comp
-L VDD #PWR028
+L VDD #PWR027
 U 1 1 466D18DB
 P 2650 1300
-F 0 "#PWR028" H 2650 1400 30  0001 C C
+F 0 "#PWR027" H 2650 1400 30  0001 C C
 F 1 "VDD" H 2650 1410 30  0000 C C
 	1    2650 1300
@@
 $EndComp
 $Comp
-L VSS #PWR029
+L VSS #PWR028
 U 1 1 466D18CA
 P 4250 2200
-F 0 "#PWR029" H 4250 2200 30  0001 C C
+F 0 "#PWR028" H 4250 2200 30  0001 C C
 F 1 "VSS" H 4250 2130 30  0000 C C
 	1    4250 2200
@@
 $EndComp
 $Comp
-L VSS #PWR030
+L VSS #PWR029
 U 1 1 466D1791
 P 10100 2500
-F 0 "#PWR030" H 10100 2500 30  0001 C C
+F 0 "#PWR029" H 10100 2500 30  0001 C C
 F 1 "VSS" H 10100 2430 30  0000 C C
 	1    10100 2500
