File: trunk/pcb/usbpicprog.sch (KiCad schematic (older format))
At the start: 46 parts, among them J1 USB_CONN, P1 CONN_5, P2 CONN_5, Q1 BS170, Q2 BS170, Q3 TSM2301CX, Q4 BS170, U1 PIC18F2550, X1 8MHz

Commit message: changed some resistor values in the schematic for better VPP behaviour, also updated the ZIF socket for I2C Eeprom
git-svn-id: https://usbpicprog.svn.sourceforge.net/svnroot/usbpicprog@852 29735491-9d32-0410-b17f-ed4c7e910dea
Parts:
- R13: value 100k -> NA
- R15: value 100k -> 1M
- R16: value 47k -> 470k

Commit message: changed some values in the PCB
git-svn-id: https://usbpicprog.svn.sourceforge.net/svnroot/usbpicprog@986 29735491-9d32-0410-b17f-ed4c7e910dea
Parts:
- removed Q4: BS170, symbol FET_N
- added Q4: BC847, symbol NPN
- D8: value 12V -> 12V or NA
- R1: value 2k2 -> 1k
Other:
- note added: "*NA means No Assembly"
