File: trunk/pcb/usbpicprog.sch (KiCad schematic (older format))
At the start: 46 parts, among them J1 USB_CONN, P1 CONN_5, P2 CONN_5, Q1 BS170, Q2 BS170, Q3 TSM2301CX, Q4 BC847, U1 PIC18F2550, X1 8MHz

Commit message: Replaced D4 with 0R resistor
Parts:
- D4: value 1n4148 -> 0R resistor
Changed lines of the file:
@@
-EESchema Schematic File Version 2  date Fri 25 Feb 2011 09:57:07 AM CET
+EESchema Schematic File Version 2  date Wed 28 Nov 2012 08:18:05 PM CET
 LIBS:power
 LIBS:usb-b
@@
 LIBS:valves
 LIBS:usbpicprog-cache
-EELAYER 24  0
+EELAYER 25  0
 EELAYER END
 $Descr A4 11700 8267
+encoding utf-8
 Sheet 1 1
 Title "Usbpicprog"
-Date "25 feb 2011"
+Date "28 nov 2012"
 Rev "0.3.2"
 Comp "usbpicprog.org"
@@
 P 5900 1400
 F 0 "D4" H 5900 1500 40  0000 C CNN
-F 1 "1n4148" H 5900 1300 40  0000 C CNN
+F 1 "0R resistor" H 5900 1300 40  0000 C CNN
 	1    5900 1400
 	1    0    0    -1

Commit message: Changed component value on PCB
Parts:
- D9: value 1n4148 -> Shottky
Changed lines of the file:
@@
-EESchema Schematic File Version 2  date Wed 28 Nov 2012 08:18:05 PM CET
+EESchema Schematic File Version 2  date Thu 21 Feb 2013 10:19:03 AM CET
 LIBS:power
 LIBS:usb-b
@@
 Sheet 1 1
 Title "Usbpicprog"
-Date "28 nov 2012"
+Date "21 feb 2013"
 Rev "0.3.2"
 Comp "usbpicprog.org"
@@
 P 8200 2050
 F 0 "D9" H 8200 2150 40  0000 C CNN
-F 1 "1n4148" H 8200 1950 40  0000 C CNN
+F 1 "Shottky" H 8200 1950 40  0000 C CNN
 	1    8200 2050
 	1    0    0    -1
