File: trunk/pcb/usbpicprog_th.sch (KiCad schematic (older format))
At the start: 37 parts, among them J1 USB_CONN, P1 CONN_5, P2 CONN_5, Q1 BS170, Q2 BS170, Q3 BS250, U1 PIC18F2550, X1 8MHz

Commit message: modified schematic for PIC24 and dsPIC33 devices, PCB not yet finished, will be released as v0.3
git-svn-id: https://usbpicprog.svn.sourceforge.net/svnroot/usbpicprog@377 29735491-9d32-0410-b17f-ed4c7e910dea
Parts:
- added R10, R11: 470, symbol R
- R4, R5: value 100 -> 470
Connections:
- wire segments 110 -> 120
Other:
- moved on the sheet: R4, R5

Commit message: copied usbpicprog.sch to usbpicprog_th.sch and translated to .brd file - still needs to be routed!
git-svn-id: https://usbpicprog.svn.sourceforge.net/svnroot/usbpicprog@708 29735491-9d32-0410-b17f-ed4c7e910dea
Parts:
- added D10: 1n4148, symbol DIODE
- added Q4: BS170, symbol FET_N
- added R12, R13, R15: 100k, symbol R
- added R14: 1k, symbol R
- added R16: 47k, symbol R
- C11: footprint 0603 -> (none)
- C2, C3: value 15p -> 22p
- D5: value LED -> WR
- D6: value LED -> RD
- D7: value LED -> ON
- R10, R11: value 470 -> 1k
- R6, R7, R8: value 150 -> 470
Connections:
- wire segments 120 -> 135
Other:
- moved on the sheet: R2, R3, R4, R5

Commit message: changed some resistor values in the schematic for better VPP behaviour, also updated the ZIF socket for I2C Eeprom
git-svn-id: https://usbpicprog.svn.sourceforge.net/svnroot/usbpicprog@852 29735491-9d32-0410-b17f-ed4c7e910dea
Parts:
- removed J1: USB_CONN, usb-b, symbol USB_CONN
- added J1: USB-B, symbol USB
- R13: value 100k -> NA
- R15: value 100k -> 1M
- R16: value 47k -> 470k

Commit message: changed some values in the PCB
git-svn-id: https://usbpicprog.svn.sourceforge.net/svnroot/usbpicprog@986 29735491-9d32-0410-b17f-ed4c7e910dea
Parts:
- removed Q4: BS170, symbol FET_N
- added Q4: BC547, symbol NPN
- D8: value 12V -> 12V or NA
- R1: value 2k2 -> 1k
Other:
- note added: "*NA means No Assembly"
